Commit message: Change folder names

File: moveit_config/config/ur.urdf (robot description, URDF)
Before this commit: robot ur, 34 links, 33 joints
Links:
- link camera_head_link: geometry collision box size=0.02505 0.09 0.025; visual mesh filename=file:///home/julian/workspace/UR3_ROS2_PICK_AND_PLACE/insta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

File: ur_description/urdf/ur.urdf (robot description, URDF)
Before this commit: robot ur, 34 links, 33 joints
Links:
- link camera_head_link: geometry collision box size=0.02505 0.09 0.025; visual mesh filename=file:///home/julian/workspace/UR3_ROS2_PICK_AND_PLACE/insta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

File: ur_description/urdf/ur_robot.urdf (robot description, URDF)
Before this commit: robot ur, 34 links, 33 joints
Links:
- link camera_head_link: geometry collision box size=0.02505 0.09 0.025; visual mesh filename=file:///home/julian/workspace/UR3_ROS2_PICK_AND_PLACE/insta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

File: ur_robot.urdf (robot description, URDF)
Before this commit: robot ur, 34 links, 33 joints
Links:
- link camera_head_link: geometry collision box size=0.02505 0.09 0.025; visual mesh filename=file:///home/julian/workspace/UR3_ROS2_PICK_AND_PLACE/insta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
